Commit message: update

File: quad_simulator/vision60_description/models/vision60/vision60.sdf.xacro (robot description, xacro)
@@ -41,4 +41,9 @@
           </mesh>
         </geometry>
+        <material>
+          <ambient>0.3 0.3 0.3 1</ambient>
+          <diffuse>0.3 0.3 0.3 1</diffuse>
+          <specular>0.3 0.3 0.3 1</specular>
+        </material>
       </visual>
       <gravity>1</gravity>
@@ -1213,4 +1218,5 @@
       </ros>
     </plugin>
+    <plugin filename="gz-sim-joint-state-publisher-system" name="gz::sim::systems::JointStatePublisher"/>
   </model>
 </sdf>
